File: Schematics/InterGas.kicad_pcb (KiCad board)
At the start: 2 copper layers, 95 x 75 mm, 28 parts, among them J1 Screw_Terminal_01x03, J2 Screw_Terminal_01x03, J3 Screw_Terminal_01x03, J4 Conn_01x03_Pin, J5 Conn_01x03_Pin, J6 Screw_Terminal_01x04, Q1 BC337, Q2 BC337, Q3 BC337, U1 WEMOS_D1_mini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

Commit message: Update Schematics
Parts:
- removed J1, J2, J3: Screw_Terminal_01x03, TerminalBlock_Altech:Altech_AK100_1x03_P5.00mm
- removed the J6 at (146.0, 82.0)
- removed the J6 at (72.5, 74.5)
- removed Q3: BC337, Package_TO_SOT_THT:TO-92_Inline
- removed R4: 4k7, Resistor_THT:R_Axial_DIN0207_L6.3mm_D2.5mm_P7.62mm_Horizontal
- removed R7, R9: 1K, Resistor_THT:R_Axial_DIN0207_L6.3mm_D2.5mm_P7.62mm_Horizontal
- removed REF** (x4): MountingHole_2.7mm_M2.5_DIN965_Pad_TopBottom, MountingHole:MountingHole_2.7mm_M2.5_DIN965_Pad_TopBottom
- removed REF**: MountingHole_2.1mm, MountingHole:MountingHole_2.1mm
- added C1: 10nF, Capacitor_THT:C_Disc_D3.0mm_W1.6mm_P2.50mm, F.Cu at (66.5, 85.2)
- added C2: 100nF, Capacitor_THT:C_Disc_D3.0mm_W1.6mm_P2.50mm, F.Cu at (64.0, 96.0)
- added H1: MountingHole, MountingHole:MountingHole_3.2mm_M3, F.Cu at (123.0, 73.5)
- added H2: MountingHole, MountingHole:MountingHole_3.2mm_M3, F.Cu at (59.0, 73.5)
- added H3: MountingHole, MountingHole:MountingHole_3.2mm_M3, F.Cu at (59.0, 151.0)
- added H4: MountingHole, MountingHole:MountingHole_3.2mm_M3, F.Cu at (123.0, 151.0)
- added J6: Screw_Terminal_01x04, TerminalBlock_Altech:Altech_AK100_1x04_P5.00mm, F.Cu at (66.5, 131.5)
- J4, J5: value Conn_01x03_Pin -> Conn_01x02_Pin; footprint Connector_PinHeader_1.00mm:PinHeader_1x03_P1.00mm_Vertical -> Connector_PinHeader_2.54mm:PinHeader_1x02_P2.54mm_Vertical
- Q1, Q2: footprint Package_TO_SOT_THT:TO-92_Inline -> Package_TO_SOT_THT:TO-92L
- U2: value LP2950-3.0_TO92 -> L78L33_TO92; footprint Package_TO_SOT_THT:TO-92_Inline -> Package_TO_SOT_THT:TO-92L
- moved U1 101.5 mm to (79.8, 77.5), turned to 0 degrees
- moved R3 53.7 mm to (101.4, 131.8), turned to 0 degrees
- moved U2 50.2 mm to (66.5, 90.0), turned to 180 degrees
- moved Q1 46.8 mm to (103.9, 137.9), turned to 0 degrees
- moved R2 42.8 mm to (101.5, 112.2)
- moved U3 42.6 mm to (101.6, 117.0)
- moved R8 36.5 mm to (113.3, 131.7)
- moved Q2 36.4 mm to (115.9, 137.7), turned to 0 degrees
- moved R6 33.1 mm to (101.4, 126.8)
- moved R5 32.0 mm to (113.4, 126.7), turned to 0 degrees
- moved J4 25.7 mm to (113.0, 88.2)
- moved R1 21.6 mm to (113.3, 112.2), turned to 0 degrees
- moved U4 19.9 mm to (113.4, 117.0), turned to 0 degrees
- moved J5 1.68 mm to (118.0, 88.2)
Connections:
- net +3V3 ESP32 renamed +3V3 ESP8266
- net +5V ESP32 renamed +5V ESP8266
- net GND ESP32 renamed GND ESP8266
- U1 pad 11: Net-(J7-Pin_4) -> unconnected-(U1-D4-Pad11)
- U1 pad 12: ESP32_LED -> unconnected-(U1-D3-Pad12)
- U1 pad 13: Net-(J7-Pin_3) -> unconnected-(U1-SDA/D2-Pad13)
- U1 pad 14: Net-(J7-Pin_2) -> unconnected-(U1-SCL/D1-Pad14)
- U1 pad 15: ESP32_Rx -> unconnected-(U1-RX-Pad15)
- U1 pad 16: ESP32_Tx -> unconnected-(U1-TX-Pad16)
- U1 pad 2: Net-(J7-Pin_1) -> unconnected-(U1-A0-Pad2)
- U1 pad 4: Net-(J7-Pin_5) -> unconnected-(U1-SCK/D5-Pad4)
- U1 pad 5: Net-(J7-Pin_6) -> ESP32_Tx
- U1 pad 6: Net-(J7-Pin_7) -> ESP32_Rx
- U1 pad 7: Net-(J7-Pin_8) -> unconnected-(U1-CS/D8-Pad7)
Routing:
- net GND Intergas: track 0.00 -> 165.3 mm
- net +5V Intergas: track 0.00 -> 128.6 mm
- net +3V3 Intergas: track 0.00 -> 99.6 mm, vias 0 -> 2
- net ESP32_Rx: track 0.00 -> 75.2 mm, vias 0 -> 1
- net +3V3 ESP8266: track 0.00 -> 66.7 mm
- net ESP32_Tx: track 0.00 -> 66.0 mm
- net GND ESP8266: track 0.00 -> 65.1 mm
- net Boiler_Tx: track 0.00 -> 53.8 mm
- net Boiler_Rx: track 0.00 -> 48.6 mm
- net Net-(Q2-C): track 0.00 -> 32.9 mm
- net Net-(Q1-C): track 0.00 -> 23.0 mm
- net GND: track 22.4 -> 0.00 mm
- net +5V ESP8266: track 0.00 -> 18.5 mm
- net Net-(Q1-B): track 0.00 -> 8.05 mm
- net Net-(Q2-B): track 0.00 -> 7.90 mm
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- added copper zone on B.Cu, net GND Intergas
- added copper zone on F.Cu, net GND Intergas
Other:
- board size 95 x 75 mm -> 72 x 86 mm
- board text added: "+5V"
- board text added: "Boiler RX ESP TX"
- board text added: "Boiler TX ESP RX"
- board text added: "GND"
- board text added: "IntergasGW V1.0"
- board text added: "Rx"
- board text added: "To Boiler"
- board text added: "To power from Boiler Close J4 and J5 and do NOT connect USB to ESP module"
- board text added: "Tx"
