File: Schematics/InterGas.kicad_sch (KiCad schematic)
At the start: 28 parts, among them J1 Screw_Terminal_01x03, J2 Screw_Terminal_01x03, J3 Screw_Terminal_01x03, J4 Conn_01x03_Pin, J5 Conn_01x03_Pin, J6 Screw_Terminal_01x04, J7 Conn_01x08_Pin, J8 Conn_01x08_Pin, J9 Conn_01x08_Pin, Q1 BC337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

Commit message: Update Schematics
Parts:
- removed C1: C_Polarized, symbol Device:C_Polarized
- removed D1: LED, symbol Device:LED
- removed J1, J2, J3: Screw_Terminal_01x03, TerminalBlock_Altech:Altech_AK100_1x03_P5.00mm, symbol Connector:Screw_Terminal_01x03
- removed J4, J5: Conn_01x03_Pin, Connector_PinHeader_1.00mm:PinHeader_1x03_P1.00mm_Vertical, symbol Connector:Conn_01x03_Pin
- removed J7, J8, J9: Conn_01x08_Pin, Connector_PinHeader_1.00mm:PinHeader_1x0`8_P1.00mm_Vertical, symbol Connector:Conn_01x08_Pin
- removed Q3: BC337, Package_TO_SOT_THT:TO-92_Inline, symbol Transistor_BJT:BC337
- removed R4: 4k7, Resistor_THT:R_Axial_DIN0207_L6.3mm_D2.5mm_P7.62mm_Horizontal, symbol Device:R_Small
- removed R7, R9: 1K, Resistor_THT:R_Axial_DIN0207_L6.3mm_D2.5mm_P7.62mm_Horizontal, symbol Device:R_Small
- added C1: 10nF, Capacitor_THT:C_Disc_D3.0mm_W1.6mm_P2.50mm, symbol Device:C
- added H1, H2, H3, H4: MountingHole, MountingHole:MountingHole_3.2mm_M3, symbol Mechanical:MountingHole
- added J4, J5: Conn_01x02_Pin, Connector_PinHeader_2.54mm:PinHeader_1x02_P2.54mm_Vertical, symbol Connector:Conn_01x02_Pin
- C2: footprint (none) -> Capacitor_THT:C_Disc_D3.0mm_W1.6mm_P2.50mm
- Q1, Q2, U2: footprint Package_TO_SOT_THT:TO-92_Inline -> Package_TO_SOT_THT:TO-92L
- R1, R2: value 1K -> 220E
- R3, R8: value 1K -> 68K
- R5, R6: value 1K -> 470E
Connections:
- net +3V3 Intergas: now also C1.1
- net +5V Intergas: now also J5.1 (Pin_1)
- net ESP32_Rx: now also U1.6 (MOSI/D7); no longer U1.15 (RX)
- net ESP32_Tx: now also U1.5 (MISO/D6); no longer U1.16 (TX)
- net GND Intergas: now also C1.2, J4.1 (Pin_1)
- net +3V3 ESP32 renamed +3V3 ESP8266
- net +5V ESP32 renamed +5V ESP8266
- net +5V ESP8266: now also J5.2 (Pin_2)
- net ESP32_LED: no longer names the net of U1.12 (D3)
- net GND ESP32 renamed GND ESP8266
- net GND ESP8266: now also J4.2 (Pin_2)
- no-connect marks 5 -> 12
Other:
- note added: "3V3 powersupply"
- note added: "Drilling holes"
- note added: "Intergas input"
- note added: "Power provided by ESP8266"
- note added: "Power provided by intergas boiler"
- note added: "To power from Boiler Close J4 and J5 and do NOT connect USB to ESP module"
- note added: "USB vs. phantom power supply"
- company: (none) -> Edwin Bontenbal
- title: (none) -> Intergas Gateway
- moved on the sheet: C2, J6, Q1, Q2, R1, R2, R3, R5, R6, R8, U1, U2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
